File: arisu.kicad_pcb (KiCad board)
At the start: 2 copper layers, 339.1 x 118.7 mm, 176 parts, among them J1 USB_B_Micro, SW1 SW_Push, SW10 SW_Push, SW11 SW_Push, SW12 SW_Push, SW13 SW_Push, SW14 SW_Push, SW15 SW_Push, SW16 SW_Push, SW17 SW_Push, SW18 SW_Push, SW19 SW_Push, SW2 SW_Push, SW20 SW_Push, SW21 SW_Push, SW22 SW_Push, SW23 SW_Push, SW24 SW_Push, SW25 SW_Push, SW26 SW_Push, SW27 SW_Push, SW28 SW_Push, SW29 SW_Push, SW3 SW_Push, SW30 SW_Push, SW31 SW_Push, SW32 SW_Push, SW33 SW_Push, SW34 SW_Push, SW35 SW_Push, SW36 SW_Push, SW37 SW_Push, SW38 SW_Push, SW39 SW_Push, SW4 SW_Push, SW40 SW_Push, SW41 SW_Push, SW42 SW_Push, SW43 SW_Push, SW44 SW_Push, SW45 SW_Push, SW46 SW_Push, SW47 SW_Push, SW48 SW_Push, SW49 SW_Push, SW5 SW_Push, SW50 SW_Push, SW51 SW_Push, SW52 SW_Push, SW53 SW_Push, SW54 SW_Push, SW55 SW_Push, SW56 SW_Push, SW57 SW_Push, SW58 SW_Push, SW59 SW_Push, SW6 SW_Push, SW60 SW_Push, SW61 SW_Push, SW62 SW_Push, SW63 SW_Push, SW64 SW_Push, SW65 SW_Push, SW66 SW_Push, SW67 SW_Push, SW7 SW_Push, SW8 SW_Push, SW9 SW_Push, U1 USBLC6-2SC6, U2 ATmega32U4-AU, Y1 Crystal_GND24

Commit message: USB-C version of the arisu
Parts:
- removed G*** (x2): LOGO, arisu:arisu-logo
- added R5: 5.1K, Resistor_SMD:R_0805_2012Metric_Pad1.15x1.40mm_HandSolder, B.Cu at (168.7, 29.5)
- added R6: 5.1K, Resistor_SMD:R_0805_2012Metric_Pad1.15x1.40mm_HandSolder, B.Cu at (182.3, 29.4)
- J1: value USB_B_Micro -> USB_C_Receptacle_USB2.0; footprint Connectors_USB:USB_Micro-B_Molex-105017-0001 -> cftkb:USB_C_GCT_USB4085
- moved C6 21.8 mm to (187.2, 43.1), turned to 0 degrees
- moved C9 20.3 mm to (180.3, 54.6)
- moved C7 13.5 mm to (167.3, 50.5), turned to 90 degrees
- moved R3 9.12 mm to (203.4, 29.2)
- moved C1 7.89 mm to (190.6, 35.2), turned to 180 degrees
- moved C2 6.48 mm to (193.5, 42.1), turned to 0 degrees
- moved C8 6.01 mm to (165.4, 41.6), turned to 180 degrees
- moved C3 5.87 mm to (181.4, 35.8), turned to 0 degrees
- moved R2 5.82 mm to (157.9, 34.5)
- moved SWR1 4.07 mm to (197.1, 28.6)
- moved R4 4.06 mm to (170.2, 55.8)
- moved C4 3.65 mm to (181.4, 33.9), turned to 0 degrees
- moved U1 3.43 mm to (164.5, 33.2)
- moved U2 3.35 mm to (175.2, 45.5)
- moved R1 2.95 mm to (157.9, 31.9)
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- renumbered PF6 to J10, PF7 to J11, VCC to J12, D+ to J13, D- to J14, GND to J15, MISO to J2, VCC to J3, SCK to J4, MOSI to J5, RES to J6, GND to J7, PF4 to J8, PF5 to J9
Connections:
- J13 pad 1: Net-(J1-Pad3) -> Net-(J1-PadA6)
- J14 pad 1: Net-(J1-Pad2) -> Net-(J1-PadA7)
- R1 pad 1: D+ -> D-
- R1 pad 2: Net-(J1-Pad3) -> Net-(J1-PadA7)
- R2 pad 1: D- -> D+
- R2 pad 2: Net-(J1-Pad2) -> Net-(J1-PadA6)
- U1 pad 1: Net-(U1-Pad1) -> (no net)
- U1 pad 3: Net-(U1-Pad3) -> (no net)
- U1 pad 4: Net-(J1-Pad2) -> Net-(J1-PadA7)
- U1 pad 6: Net-(J1-Pad3) -> Net-(J1-PadA6)
- U2 pad 42: Net-(U2-Pad42) -> (no net)
Routing:
- net Net-(J1-PadA6): track 0.00 -> 55.3 mm, vias 0 -> 2
- net VCC: track 205.4 -> 256.8 mm, vias 9 -> 10
- net Net-(J1-Pad3): track 47.8 -> 0.00 mm
- net Net-(J1-Pad2): track 45.1 -> 0.00 mm
- net Net-(J1-PadA7): track 0.00 -> 44.2 mm, vias 0 -> 1
- net /col12: track 249.0 -> 278.9 mm
- net /col11: track 230.6 -> 257.4 mm
- net XTAL1: track 13.1 -> 34.4 mm
- net /row1: track 384.1 -> 371.7 mm
- net /MOSI: track 39.7 -> 49.4 mm
- net GND: track 71.6 -> 80.4 mm, vias 12 -> 7
- net /row0: track 328.0 -> 320.6 mm
- net Net-(J1-PadA5): track 0.00 -> 6.92 mm
- net /col3: track 133.3 -> 140.1 mm, vias 0 -> 1
- net Net-(J1-PadB5): track 0.00 -> 6.53 mm
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Other:
- board text added: "Erladion Design Rev 1.2"
- board text removed: "Fate Design Rev 1.1"

Commit message: First commit with arisu using a stm32f411 and usb-c
Parts:
- removed J10: PF6, Pin_Headers:Pin_Header_Straight_1x01_Pitch2.54mm
- removed J11: PF7, Pin_Headers:Pin_Header_Straight_1x01_Pitch2.54mm
- removed J6: RES, Pin_Headers:Pin_Header_Straight_1x01_Pitch2.54mm
- removed J7: GND, Pin_Headers:Pin_Header_Straight_1x01_Pitch2.54mm
- removed J8: PF4, Pin_Headers:Pin_Header_Straight_1x01_Pitch2.54mm
- removed J9: PF5, Pin_Headers:Pin_Header_Straight_1x01_Pitch2.54mm
- added C10: 100nF, Capacitor_SMD:C_0805_2012Metric_Pad1.15x1.40mm_HandSolder, B.Cu at (181.8, 55.5)
- added C11: 100nF, Capacitor_SMD:C_0805_2012Metric_Pad1.15x1.40mm_HandSolder, B.Cu at (180.8, 58.8)
- added C12: 100nF, Capacitor_SMD:C_0805_2012Metric_Pad1.15x1.40mm_HandSolder, B.Cu at (162.8, 62.5)
- added C13: 100nF, Capacitor_SMD:C_0805_2012Metric_Pad1.15x1.40mm_HandSolder, B.Cu at (180.6, 40.6)
- added C14: 100nF, Capacitor_SMD:C_0805_2012Metric_Pad1.15x1.40mm_HandSolder, B.Cu at (168.2, 41.8)
- added C15: 100nF, Capacitor_SMD:C_0805_2012Metric_Pad1.15x1.40mm_HandSolder, B.Cu at (168.6, 57.9)
- added C16: 1.0uF, Capacitor_SMD:C_0805_2012Metric_Pad1.15x1.40mm_HandSolder, B.Cu at (163.9, 30.1)
- added L1: 10uH, Inductor_SMD:L_0805_2012Metric_Pad1.15x1.40mm_HandSolder, B.Cu at (165.4, 58.9)
- added SW68: SW_Push, Button_Switch_SMD:SW_SPST_TL3342, B.Cu at (167.7, 68.0)
- added U5: STM32F411RETx, Package_QFP:LQFP-64_10x10mm_P0.5mm, B.Cu at (174.7, 48.7)
- added Y2: Crystal_Small, Crystal:Crystal_SMD_MicroCrystal_CC7V-T1A-2Pin_3.2x1.5mm_HandSoldering, B.Cu at (180.1, 63.8)
- C1, C2: value 22pF -> 12pF; footprint Capacitors_SMD:C_0805_HandSoldering -> Capacitor_SMD:C_0805_2012Metric_Pad1.15x1.40mm_HandSolder
- C3: value 10uF -> 100nF; footprint Capacitors_SMD:C_0805_HandSoldering -> Capacitor_SMD:C_0805_2012Metric_Pad1.15x1.40mm_HandSolder
- C4: value 1uF (±10%) -> 1.0uF; footprint Capacitors_SMD:C_0805_HandSoldering -> Capacitor_SMD:C_0805_2012Metric_Pad1.15x1.40mm_HandSolder
- C5: value 1uF -> 15pF; footprint Capacitors_SMD:C_0805_HandSoldering -> Capacitor_SMD:C_0805_2012Metric_Pad1.15x1.40mm_HandSolder
- C6: value 0.1uF -> 15pF; footprint Capacitors_SMD:C_0805_HandSoldering -> Capacitor_SMD:C_0805_2012Metric_Pad1.15x1.40mm_HandSolder
- C7, C9: value 0.1uF -> 100nF; footprint Capacitors_SMD:C_0805_HandSoldering -> Capacitor_SMD:C_0805_2012Metric_Pad1.15x1.40mm_HandSolder
- C8: value 0.1uF -> 2.2uF; footprint Capacitors_SMD:C_0805_HandSoldering -> Capacitor_SMD:C_0805_2012Metric_Pad1.15x1.40mm_HandSolder
- J12, J13, J14, J15: footprint Pin_Headers:Pin_Header_Straight_1x01_Pitch2.54mm -> Connector_PinHeader_2.54mm:PinHeader_1x01_P2.54mm_Vertical
- J2: value MISO -> 3.3V; footprint Pin_Headers:Pin_Header_Straight_1x01_Pitch2.54mm -> Connector_PinHeader_2.54mm:PinHeader_1x01_P2.54mm_Vertical
- J3: value VCC -> SWDIO; footprint Pin_Headers:Pin_Header_Straight_1x01_Pitch2.54mm -> Connector_PinHeader_2.54mm:PinHeader_1x01_P2.54mm_Vertical
- J4: value SCK -> SWCLK; footprint Pin_Headers:Pin_Header_Straight_1x01_Pitch2.54mm -> Connector_PinHeader_2.54mm:PinHeader_1x01_P2.54mm_Vertical
- J5: value MOSI -> GND; footprint Pin_Headers:Pin_Header_Straight_1x01_Pitch2.54mm -> Connector_PinHeader_2.54mm:PinHeader_1x01_P2.54mm_Vertical
- R1, R2: value 22 -> 10; footprint Resistors_SMD:R_0805_HandSoldering -> Resistor_SMD:R_0805_2012Metric_Pad1.15x1.40mm_HandSolder
- R3, R4: footprint Resistors_SMD:R_0805_HandSoldering -> Resistor_SMD:R_0805_2012Metric_Pad1.15x1.40mm_HandSolder
- SWR1: footprint Buttons_Switches_SMD:SW_SPST_TL3342 -> Button_Switch_SMD:SW_SPST_TL3342
- U2: value ATmega32U4-AU -> ADP7142AUJZ-3.3; footprint Housings_QFP:TQFP-44_10x10mm_Pitch0.8mm -> Package_TO_SOT_SMD:TSOT-23-5
- Y1: footprint Crystals:Crystal_SMD_SeikoEpson_FA238-4pin_3.2x2.5mm_HandSoldering -> Crystal:Crystal_SMD_SeikoEpson_TSX3225-4Pin_3.2x2.5mm_HandSoldering
- moved J3 69.9 mm to (148.3, 26.5), turned to 180 degrees
- moved J2 67.4 mm to (153.3, 26.4), turned to 180 degrees
- moved J5 67.4 mm to (145.7, 26.5), turned to 180 degrees
- moved J4 64.8 mm to (150.8, 26.5), turned to 180 degrees
- moved J15 60.0 mm to (203.8, 26.9), turned to 180 degrees
- moved J13 54.9 mm to (201.2, 26.9), turned to 180 degrees
- moved J14 49.9 mm to (198.7, 26.9), turned to 180 degrees
- moved J12 44.8 mm to (196.2, 26.9), turned to 180 degrees
- moved C1 35.4 mm to (174.4, 66.7)
- moved C5 30.0 mm to (183.7, 62.5)
- moved Y1 28.9 mm to (174.5, 62.5), turned to 90 degrees
- moved C2 25.0 mm to (174.6, 58.4), turned to 180 degrees
- moved C6 22.2 mm to (183.7, 65.1)
- moved R1 21.6 mm to (178.9, 36.8)
- moved R2 21.0 mm to (178.9, 34.8)
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Connections:
- C1 pad 2: XTAL1 -> OSC_OUT
- C2 pad 1: XTAL2 -> OSC_IN
- C3 pad 1: VCC -> GND
- C3 pad 2: GND -> VCC
- C4 pad 1: Net-(C4-Pad1) -> GND
- C4 pad 2: GND -> VCC
- C5 pad 1: VCC -> GND
- C5 pad 2: GND -> OSC32_IN
- C6 pad 1: VCC -> OSC32_OUT
- C7 pad 1: VCC -> GND
- C7 pad 2: GND -> 3.3V
- C8 pad 1: VCC -> Net-(C8-Pad1)
- C9 pad 1: VCC -> GND
- C9 pad 2: GND -> 3.3V
- D1 pad 1: /row0 -> row0
- D10 pad 1: /row0 -> row0
- D11 pad 1: /row1 -> row1
- D12 pad 1: /row2 -> row2
- D13 pad 1: /row3 -> row3
- D14 pad 1: /row4 -> row4
- D15 pad 1: /row0 -> row0
- D16 pad 1: /row1 -> row1
- D17 pad 1: /row2 -> row2
- D18 pad 1: /row3 -> row3
- D19 pad 1: /row0 -> row0
- D2 pad 1: /row1 -> row1
- D20 pad 1: /row1 -> row1
- D21 pad 1: /row2 -> row2
- D22 pad 1: /row3 -> row3
- D23 pad 1: /row4 -> row4
- D24 pad 1: /row0 -> row0
- D25 pad 1: /row1 -> row1
- D26 pad 1: /row2 -> row2
- D27 pad 1: /row3 -> row3
- D28 pad 1: /row4 -> row4
- D29 pad 1: /row0 -> row0
- D3 pad 1: /row2 -> row2
- D30 pad 1: /row1 -> row1
- D31 pad 1: /row2 -> row2
- D32 pad 1: /row3 -> row3
- D33 pad 1: /row0 -> row0
- D34 pad 1: /row1 -> row1
- D35 pad 1: /row2 -> row2
- D36 pad 1: /row3 -> row3
- D37 pad 1: /row4 -> row4
- D38 pad 1: /row0 -> row0
- D39 pad 1: /row1 -> row1
- D4 pad 1: /row3 -> row3
- D40 pad 1: /row2 -> row2
- D41 pad 1: /row3 -> row3
- D42 pad 1: /row0 -> row0
- D43 pad 1: /row1 -> row1
- D44 pad 1: /row2 -> row2
- D45 pad 1: /row3 -> row3
- D46 pad 1: /row4 -> row4
- D47 pad 1: /row0 -> row0
- D48 pad 1: /row1 -> row1
- D49 pad 1: /row2 -> row2
- D5 pad 1: /row4 -> row4
- D50 pad 1: /row3 -> row3
- D51 pad 1: /row0 -> row0
- D52 pad 1: /row1 -> row1
- D53 pad 1: /row2 -> row2
- D54 pad 1: /row3 -> row3
- D55 pad 1: /row0 -> row0
- D56 pad 1: /row1 -> row1
- D57 pad 1: /row2 -> row2
- D58 pad 1: /row4 -> row4
- D59 pad 1: /row0 -> row0
- D6 pad 1: /row0 -> row0
- D60 pad 1: /row1 -> row1
- D61 pad 1: /row3 -> row3
- D62 pad 1: /row4 -> row4
- D63 pad 1: /row0 -> row0
- D64 pad 1: /row1 -> row1
- D65 pad 1: /row2 -> row2
- D66 pad 1: /row3 -> row3
- D67 pad 1: /row4 -> row4
- D7 pad 1: /row1 -> row1
- D8 pad 1: /row2 -> row2
- D9 pad 1: /row3 -> row3
- J2 pad 1: /MISO -> 3.3V
- J3 pad 1: VCC -> SWDIO
- J4 pad 1: /SCK -> SWCLK
- J5 pad 1: /MOSI -> GND
- R3 pad 1: VCC -> GND
- R3 pad 2: /~RES~ -> Net-(R3-Pad2)
- SW1 pad 1: /col0 -> col0
- SW10 pad 1: /col2 -> col2
- SW11 pad 1: /col2 -> col2
- SW12 pad 1: /col2 -> col2
- SW13 pad 1: /col2 -> col2
- SW14 pad 1: /col2 -> col2
- SW15 pad 1: /col3 -> col3
- SW16 pad 1: /col3 -> col3
- SW17 pad 1: /col3 -> col3
- SW18 pad 1: /col3 -> col3
- SW19 pad 1: /col4 -> col4
- SW2 pad 1: /col0 -> col0
- SW20 pad 1: /col4 -> col4
- SW21 pad 1: /col4 -> col4
- SW22 pad 1: /col4 -> col4
- SW23 pad 1: /col4 -> col4
- SW24 pad 1: /col5 -> col5
- SW25 pad 1: /col5 -> col5
- SW26 pad 1: /col5 -> col5
- SW27 pad 1: /col5 -> col5
- SW28 pad 1: /col5 -> col5
- SW29 pad 1: /col6 -> col6
- SW3 pad 1: /col0 -> col0
- SW30 pad 1: /col6 -> col6
- SW31 pad 1: /col6 -> col6
- SW32 pad 1: /col6 -> col6
- SW33 pad 1: /SCK -> col7
- SW34 pad 1: /SCK -> col7
- SW35 pad 1: /SCK -> col7
- SW36 pad 1: /SCK -> col7
- SW37 pad 1: /SCK -> col7
- SW38 pad 1: /col8 -> col8
- SW39 pad 1: /col8 -> col8
- SW4 pad 1: /col0 -> col0
- SW40 pad 1: /col8 -> col8
- SW41 pad 1: /col8 -> col8
- SW42 pad 1: /col9 -> col9
- SW43 pad 1: /col9 -> col9
- SW44 pad 1: /col9 -> col9
- SW45 pad 1: /col9 -> col9
- SW46 pad 1: /col9 -> col9
- SW47 pad 1: /col10 -> col10
- SW48 pad 1: /col10 -> col10
- SW49 pad 1: /col10 -> col10
- SW5 pad 1: /col0 -> col0
- SW50 pad 1: /col10 -> col10
- SW51 pad 1: /col11 -> col11
- SW52 pad 1: /col11 -> col11
- SW53 pad 1: /col11 -> col11
- SW54 pad 1: /col11 -> col11
- SW55 pad 1: /col12 -> col12
- SW56 pad 1: /col12 -> col12
- SW57 pad 1: /col12 -> col12
- SW58 pad 1: /col12 -> col12
- SW59 pad 1: /col13 -> col13
- SW6 pad 1: /col1 -> col1
- SW60 pad 1: /col13 -> col13
- SW61 pad 1: /col13 -> col13
- SW62 pad 1: /col13 -> col13
- SW63 pad 1: /MISO -> col14
- SW64 pad 1: /MISO -> col14
- SW65 pad 1: /MISO -> col14
- SW66 pad 1: /MISO -> col14
- SW67 pad 1: /MISO -> col14
- SW7 pad 1: /col1 -> col1
- SW8 pad 1: /col1 -> col1
- SW9 pad 1: /col1 -> col1
- SWR1 pad 1: GND -> 3.3V
- SWR1 pad 2: /~RES~ -> Net-(R3-Pad2)
- U2 pad 1: /col2 -> VCC
- U2 pad 2: VCC -> GND
- U2 pad 3: D- -> VCC
- U2 pad 4: D+ -> GND
- U2 pad 5: GND -> 3.3V
- Y1 pad 1: XTAL1 -> OSC_OUT
- Y1 pad 3: XTAL2 -> OSC_IN
Routing:
- net row4: track 0.00 -> 432.5 mm, vias 0 -> 2
- net /row4: track 429.1 -> 0.00 mm, vias 2 -> 0
- net /row3: track 426.5 -> 0.00 mm, vias 2 -> 0
- net row3: track 0.00 -> 423.1 mm, vias 0 -> 2
- net /row2: track 396.4 -> 0.00 mm, vias 4 -> 0
- net row2: track 0.00 -> 393.7 mm, vias 0 -> 2
- net /row1: track 371.7 -> 0.00 mm, vias 4 -> 0
- net row1: track 0.00 -> 369.7 mm, vias 0 -> 2
- net row0: track 0.00 -> 323.1 mm
- net /row0: track 320.6 -> 0.00 mm, vias 4 -> 0
- net col14: track 0.00 -> 279.2 mm, vias 0 -> 1
- net /col12: track 278.9 -> 0.00 mm
- net /MISO: track 276.9 -> 0.00 mm, vias 1 -> 0
- net /col13: track 264.4 -> 0.00 mm
- net /col11: track 257.4 -> 0.00 mm
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Other:
- rule via_min_size: 0.7 -> 0.4
- board text added: "Erladion Arisu Rev 0.4"
- board text removed: "Erladion Design Rev 1.2"
