File: arisu.kicad_pcb (KiCad board)
At the start: 2 copper layers, 339.1 x 118.7 mm, 176 parts, among them J1 USB_C_Receptacle_USB2.0, J10 PF6, J11 PF7, J12 VCC, J13 D+, J14 D-, J15 GND, J2 MISO, J3 VCC, J4 SCK, J5 MOSI, J6 RES, J7 GND, J8 PF4, J9 PF5, SW1 SW_Push, SW10 SW_Push, SW11 SW_Push, SW12 SW_Push, SW13 SW_Push, SW14 SW_Push, SW15 SW_Push, SW16 SW_Push, SW17 SW_Push, SW18 SW_Push, SW19 SW_Push, SW2 SW_Push, SW20 SW_Push, SW21 SW_Push, SW22 SW_Push, SW23 SW_Push, SW24 SW_Push, SW25 SW_Push, SW26 SW_Push, SW27 SW_Push, SW28 SW_Push, SW29 SW_Push, SW3 SW_Push, SW30 SW_Push, SW31 SW_Push, SW32 SW_Push, SW33 SW_Push, SW34 SW_Push, SW35 SW_Push, SW36 SW_Push, SW37 SW_Push, SW38 SW_Push, SW39 SW_Push, SW4 SW_Push, SW40 SW_Push, SW41 SW_Push, SW42 SW_Push, SW43 SW_Push, SW44 SW_Push, SW45 SW_Push, SW46 SW_Push, SW47 SW_Push, SW48 SW_Push, SW49 SW_Push, SW5 SW_Push, SW50 SW_Push, SW51 SW_Push, SW52 SW_Push, SW53 SW_Push, SW54 SW_Push, SW55 SW_Push, SW56 SW_Push, SW57 SW_Push, SW58 SW_Push, SW59 SW_Push, SW6 SW_Push, SW60 SW_Push, SW61 SW_Push, SW62 SW_Push, SW63 SW_Push, SW64 SW_Push, SW65 SW_Push, SW66 SW_Push, SW67 SW_Push, SW7 SW_Push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

Commit message: Update references to show values
Parts:
- Atmega 32u4: renamed from U2
- renumbered C9 to 0.1uF, C6 to 0.1uF, C7 to 0.1uF, C8 to 0.1uF, R3 to 10K, R4 to 10K, C3 to 10uF, C4 to 1uF, C5 to 1uF, R1 to 22, R2 to 22, C1 to 22pF, C2 to 22pF, R6 to 5.1K, R5 to 5.1K, J13 to D+, J14 to D-, J7 to GND, J15 to GND, J2 to MISO, J5 to MOSI, J8 to PF4, J9 to PF5, J10 to PF6, J11 to PF7, J6 to RES, SWR1 to RESET, J4 to SCK, U1 to USBLC6, J3 to VCC, J12 to VCC
